Commit message: Fix URDF joint8/9

File: robotis_mini/urdf/robotis_mini.urdf (robot description, URDF)
Before this commit: robot mini, 17 links, 16 joints
Joints:
- removed joint Joint_8
- added joint Joint_08: type continuous, parent Body, child L_leg_01, origin xyz=0 0.0720000000000003 0.0239999999999996 rpy=1.56326728402668 0 1.57079632679526, axis 0 0.00752897163592653 -0.999971656891387
- joint Joint_09: type fixed -> continuous

Commit message: Fix joint 9 normal vector

File: robotis_mini/urdf/robotis_mini.urdf (robot description, URDF)
Before this commit: robot mini, 17 links, 16 joints
Joints:
- joint Joint_09: axis 0 0 0 -> 0 0 1

Commit message: Fix mesh location in package (not TA's original location)

File: robotis_mini/urdf/robotis_mini.urdf (robot description, URDF)
Before this commit: robot mini, 17 links, 16 joints
Links:
- link Body: geometry collision mesh filename=package://meshes/Body.STL; visual mesh filename=package://meshes/Body.STL
- link L_arm_01: geometry collision mesh filename=package://meshes/L_arm_01.STL; visual mesh filename=package://meshes/L_arm_01.STL
- link L_arm_02: geometry collision mesh filename=package://meshes/L_arm_02.STL; visual mesh filename=package://meshes/L_arm_02.STL
- link L_arm_03: geometry collision mesh filename=package://meshes/L_arm_03.STL; visual mesh filename=package://meshes/L_arm_03.STL
- link L_leg_01: geometry collision mesh filename=package://meshes/L_leg_01.STL; visual mesh filename=package://meshes/L_leg_01.STL
- link L_leg_02: geometry collision mesh filename=package://meshes/L_leg_02.STL; visual mesh filename=package://meshes/L_leg_02.STL
- link L_leg_03: geometry collision mesh filename=package://meshes/L_leg_03.STL; visual mesh filename=package://meshes/L_leg_03.STL
- link L_leg_04: geometry collision mesh filename=package://meshes/L_leg_04.STL; visual mesh filename=package://meshes/L_leg_04.STL
- link L_leg_05: geometry collision mesh filename=package://meshes/L_leg_05.STL; visual mesh filename=package://meshes/L_leg_05.STL
- link R_Leg_02: geometry collision mesh filename=package://meshes/R_Leg_02.STL; visual mesh filename=package://meshes/R_Leg_02.STL
- link R_arm_01: geometry collision mesh filename=package://meshes/R_arm_01.STL; visual mesh filename=package://meshes/R_arm_01.STL
- link R_arm_02: geometry collision mesh filename=package://meshes/R_arm_02.STL; visual mesh filename=package://meshes/R_arm_02.STL
- link R_arm_03: geometry collision mesh filename=package://meshes/R_arm_03.STL; visual mesh filename=package://meshes/R_arm_03.STL
- link R_leg_01: geometry collision mesh filename=package://meshes/R_leg_01.STL; visual mesh filename=package://meshes/R_leg_01.STL
- link R_leg_03: geometry collision mesh filename=package://meshes/R_leg_03.STL; visual mesh filename=package://meshes/R_leg_03.STL
- link R_leg_04: geometry collision mesh filename=package://meshes/R_leg_04.STL; visual mesh filename=package://meshes/R_leg_04.STL
- link R_leg_05: geometry collision mesh filename=package://meshes/R_leg_05.STL; visual mesh filename=package://meshes/R_leg_05.STL

Commit message: Fix mesh location and change engine to bullet.

File: robotis_mini/urdf/robotis_mini.urdf (robot description, URDF)
Before this commit: robot mini, 17 links, 16 joints
Links:
- link Body: geometry collision mesh filename=package://robotis_mini/meshes/Body.STL; visual mesh filename=package://robotis_mini/meshes/Body.STL
- link L_arm_01: geometry collision mesh filename=package://robotis_mini/meshes/L_arm_01.STL; visual mesh filename=package://robotis_mini/meshes/L_arm_01.STL
- link L_arm_02: geometry collision mesh filename=package://robotis_mini/meshes/L_arm_02.STL; visual mesh filename=package://robotis_mini/meshes/L_arm_02.STL
- link L_arm_03: geometry collision mesh filename=package://robotis_mini/meshes/L_arm_03.STL; visual mesh filename=package://robotis_mini/meshes/L_arm_03.STL
- link L_leg_01: geometry collision mesh filename=package://robotis_mini/meshes/L_leg_01.STL; visual mesh filename=package://robotis_mini/meshes/L_leg_01.STL
- link L_leg_02: geometry collision mesh filename=package://robotis_mini/meshes/L_leg_02.STL; visual mesh filename=package://robotis_mini/meshes/L_leg_02.STL
- link L_leg_03: geometry collision mesh filename=package://robotis_mini/meshes/L_leg_03.STL; visual mesh filename=package://robotis_mini/meshes/L_leg_03.STL
- link L_leg_04: geometry collision mesh filename=package://robotis_mini/meshes/L_leg_04.STL; visual mesh filename=package://robotis_mini/meshes/L_leg_04.STL
- link L_leg_05: geometry collision mesh filename=package://robotis_mini/meshes/L_leg_05.STL; visual mesh filename=package://robotis_mini/meshes/L_leg_05.STL
- link R_Leg_02: geometry collision mesh filename=package://robotis_mini/meshes/R_Leg_02.STL; visual mesh filename=package://robotis_mini/meshes/R_Leg_02.STL
- link R_arm_01: geometry collision mesh filename=package://robotis_mini/meshes/R_arm_01.STL; visual mesh filename=package://robotis_mini/meshes/R_arm_01.STL
- link R_arm_02: geometry collision mesh filename=package://robotis_mini/meshes/R_arm_02.STL; visual mesh filename=package://robotis_mini/meshes/R_arm_02.STL
- link R_arm_03: geometry collision mesh filename=package://robotis_mini/meshes/R_arm_03.STL; visual mesh filename=package://robotis_mini/meshes/R_arm_03.STL
- link R_leg_01: geometry collision mesh filename=package://robotis_mini/meshes/R_leg_01.STL; visual mesh filename=package://robotis_mini/meshes/R_leg_01.STL
- link R_leg_03: geometry collision mesh filename=package://robotis_mini/meshes/R_leg_03.STL; visual mesh filename=package://robotis_mini/meshes/R_leg_03.STL
- link R_leg_04: geometry collision mesh filename=package://robotis_mini/meshes/R_leg_04.STL; visual mesh filename=package://robotis_mini/meshes/R_leg_04.STL
- link R_leg_05: geometry collision mesh filename=package://robotis_mini/meshes/R_leg_05.STL; visual mesh filename=package://robotis_mini/meshes/R_leg_05.STL

Commit message: Add no-intertia patch. Fix hardware non-default gear ratio.

File: robotis_mini/urdf/robotis_mini.urdf (robot description, URDF)
Before this commit: robot mini, 17 links, 16 joints
Links:
- added link world_link
Joints:
- added joint world_to_body: type fixed, parent world_link, child Body
