Commit message: Make the sim package purely for simulation and no contact with hardware.

File: robotis_mini_sim/urdf/robotis_mini.urdf (robot description, URDF)
Before this commit: robot mini, 18 links, 17 joints
Links:
- link Body: geometry collision mesh filename=package://robotis_mini_sim/meshes/Body.STL; visual mesh filename=package://robotis_mini_sim/meshes/Body.STL
- link L_arm_01: geometry collision mesh filename=package://robotis_mini_sim/meshes/L_arm_01.STL; visual mesh filename=package://robotis_mini_sim/meshes/L_arm_01.STL
- link L_arm_02: geometry collision mesh filename=package://robotis_mini_sim/meshes/L_arm_02.STL; visual mesh filename=package://robotis_mini_sim/meshes/L_arm_02.STL
- link L_arm_03: geometry collision mesh filename=package://robotis_mini_sim/meshes/L_arm_03.STL; visual mesh filename=package://robotis_mini_sim/meshes/L_arm_03.STL
- link L_leg_01: geometry collision mesh filename=package://robotis_mini_sim/meshes/L_leg_01.STL; visual mesh filename=package://robotis_mini_sim/meshes/L_leg_01.STL
- link L_leg_02: geometry collision mesh filename=package://robotis_mini_sim/meshes/L_leg_02.STL; visual mesh filename=package://robotis_mini_sim/meshes/L_leg_02.STL
- link L_leg_03: geometry collision mesh filename=package://robotis_mini_sim/meshes/L_leg_03.STL; visual mesh filename=package://robotis_mini_sim/meshes/L_leg_03.STL
- link L_leg_04: geometry collision mesh filename=package://robotis_mini_sim/meshes/L_leg_04.STL; visual mesh filename=package://robotis_mini_sim/meshes/L_leg_04.STL
- link L_leg_05: geometry collision mesh filename=package://robotis_mini_sim/meshes/L_leg_05.STL; visual mesh filename=package://robotis_mini_sim/meshes/L_leg_05.STL
- link R_Leg_02: geometry collision mesh filename=package://robotis_mini_sim/meshes/R_Leg_02.STL; visual mesh filename=package://robotis_mini_sim/meshes/R_Leg_02.STL
- link R_arm_01: geometry collision mesh filename=package://robotis_mini_sim/meshes/R_arm_01.STL; visual mesh filename=package://robotis_mini_sim/meshes/R_arm_01.STL
- link R_arm_02: geometry collision mesh filename=package://robotis_mini_sim/meshes/R_arm_02.STL; visual mesh filename=package://robotis_mini_sim/meshes/R_arm_02.STL
- link R_arm_03: geometry collision mesh filename=package://robotis_mini_sim/meshes/R_arm_03.STL; visual mesh filename=package://robotis_mini_sim/meshes/R_arm_03.STL
- link R_leg_01: geometry collision mesh filename=package://robotis_mini_sim/meshes/R_leg_01.STL; visual mesh filename=package://robotis_mini_sim/meshes/R_leg_01.STL
- link R_leg_03: geometry collision mesh filename=package://robotis_mini_sim/meshes/R_leg_03.STL; visual mesh filename=package://robotis_mini_sim/meshes/R_leg_03.STL
- link R_leg_04: geometry collision mesh filename=package://robotis_mini_sim/meshes/R_leg_04.STL; visual mesh filename=package://robotis_mini_sim/meshes/R_leg_04.STL
- link R_leg_05: geometry collision mesh filename=package://robotis_mini_sim/meshes/R_leg_05.STL; visual mesh filename=package://robotis_mini_sim/meshes/R_leg_05.STL

Commit message: Revert to dartsim. Provide decimated mesh for collision.

File: robotis_mini_sim/urdf/robotis_mini.urdf (robot description, URDF)
Before this commit: robot mini, 18 links, 17 joints
Links:
- link Body: geometry collision mesh filename=package://robotis_mini_sim/meshes/Body_d.STL; visual mesh filename=package://robotis_mini_sim/meshes/Body.STL
- link L_arm_01: geometry collision mesh filename=package://robotis_mini_sim/meshes/L_arm_01_d.STL; visual mesh filename=package://robotis_mini_sim/meshes/L_arm_01.STL
- link L_arm_02: geometry collision mesh filename=package://robotis_mini_sim/meshes/L_arm_02_d.STL; visual mesh filename=package://robotis_mini_sim/meshes/L_arm_02.STL
- link L_arm_03: geometry collision mesh filename=package://robotis_mini_sim/meshes/L_arm_03_d.STL; visual mesh filename=package://robotis_mini_sim/meshes/L_arm_03.STL
- link L_leg_01: geometry collision mesh filename=package://robotis_mini_sim/meshes/L_leg_01_d.STL; visual mesh filename=package://robotis_mini_sim/meshes/L_leg_01.STL
- link L_leg_02: geometry collision mesh filename=package://robotis_mini_sim/meshes/L_leg_02_d.STL; visual mesh filename=package://robotis_mini_sim/meshes/L_leg_02.STL
- link L_leg_03: geometry collision mesh filename=package://robotis_mini_sim/meshes/L_leg_03_d.STL; visual mesh filename=package://robotis_mini_sim/meshes/L_leg_03.STL
- link L_leg_04: geometry collision mesh filename=package://robotis_mini_sim/meshes/L_leg_04_d.STL; visual mesh filename=package://robotis_mini_sim/meshes/L_leg_04.STL
- link L_leg_05: geometry collision mesh filename=package://robotis_mini_sim/meshes/L_leg_05_d.STL; visual mesh filename=package://robotis_mini_sim/meshes/L_leg_05.STL
- link R_Leg_02: geometry collision mesh filename=package://robotis_mini_sim/meshes/R_Leg_02_d.STL; visual mesh filename=package://robotis_mini_sim/meshes/R_Leg_02.STL
- link R_arm_01: geometry collision mesh filename=package://robotis_mini_sim/meshes/R_arm_01_d.STL; visual mesh filename=package://robotis_mini_sim/meshes/R_arm_01.STL
- link R_arm_02: geometry collision mesh filename=package://robotis_mini_sim/meshes/R_arm_02_d.STL; visual mesh filename=package://robotis_mini_sim/meshes/R_arm_02.STL
- link R_arm_03: geometry collision mesh filename=package://robotis_mini_sim/meshes/R_arm_03_d.STL; visual mesh filename=package://robotis_mini_sim/meshes/R_arm_03.STL
- link R_leg_01: geometry collision mesh filename=package://robotis_mini_sim/meshes/R_leg_01_d.STL; visual mesh filename=package://robotis_mini_sim/meshes/R_leg_01.STL
- link R_leg_03: geometry collision mesh filename=package://robotis_mini_sim/meshes/R_leg_03_d.STL; visual mesh filename=package://robotis_mini_sim/meshes/R_leg_03.STL
- link R_leg_04: geometry collision mesh filename=package://robotis_mini_sim/meshes/R_leg_04_d.STL; visual mesh filename=package://robotis_mini_sim/meshes/R_leg_04.STL
- link R_leg_05: geometry collision mesh filename=package://robotis_mini_sim/meshes/R_leg_05_d.STL; visual mesh filename=package://robotis_mini_sim/meshes/R_leg_05.STL
