Commit message: Update urdf installation path and default camera pose (doesn't seem to wrok)

File: robotis_mini_model/urdf/common.urdf.xacro (robot description, xacro)
@@ -92,5 +92,5 @@
         <geometry>
           <mesh
-            filename="package://robotis_mini_description/meshes/Body.STL" />
+            filename="package://robotis_mini_model/meshes/Body.STL" />
         </geometry>
         <material
@@ -106,5 +106,5 @@
         <geometry>
           <mesh
-            filename="package://robotis_mini_description/meshes/Body.STL" />
+            filename="package://robotis_mini_model/meshes/Body.STL" />
         </geometry>
       </collision>
@@ -145,5 +145,5 @@
         <origin xyz="0 0 0" rpy="0 0 0" />
         <geometry>
-          <mesh filename="package://robotis_mini_description/meshes/DMF-B01(W).stl" scale="${STL_SCALE}" />
+          <mesh filename="package://robotis_mini_model/meshes/DMF-B01(W).stl" scale="${STL_SCALE}" />
         </geometry>
         <material name="White" />
@@ -159,5 +159,5 @@
       <collision>
         <geometry>
-          <mesh filename="package://robotis_mini_description/meshes/DMF-B01(W)_s.stl" scale="${STL_SCALE}" />
+          <mesh filename="package://robotis_mini_model/meshes/DMF-B01(W)_s.stl" scale="${STL_SCALE}" />
         </geometry>
       </collision>
@@ -175,5 +175,5 @@
         <origin xyz="0 0 0" rpy="0 0 0" />
         <geometry>
-          <mesh filename="package://robotis_mini_description/meshes/DMB-B02(W).stl" scale="${STL_SCALE}" />
+          <mesh filename="package://robotis_mini_model/meshes/DMB-B02(W).stl" scale="${STL_SCALE}" />
         </geometry>
         <material name="White" />
@@ -189,5 +189,5 @@
       <collision>
         <geometry>
-          <mesh filename="package://robotis_mini_description/meshes/DMB-B02(W)_s.stl" scale="${STL_SCALE}" />
+          <mesh filename="package://robotis_mini_model/meshes/DMB-B02(W)_s.stl" scale="${STL_SCALE}" />
         </geometry>
       </collision>
@@ -205,5 +205,5 @@
         <origin xyz="0 0 0" rpy="0 0 0" />
         <geometry>
-          <mesh filename="package://robotis_mini_description/meshes/DMF-B03(W).stl" scale="${STL_SCALE}" />
+          <mesh filename="package://robotis_mini_model/meshes/DMF-B03(W).stl" scale="${STL_SCALE}" />
         </geometry>
         <material name="White" />
@@ -219,5 +219,5 @@
       <collision>
         <geometry>
-          <mesh filename="package://robotis_mini_description/meshes/DMF-B03(W)_s.stl" scale="${STL_SCALE}" />
+          <mesh filename="package://robotis_mini_model/meshes/DMF-B03(W)_s.stl" scale="${STL_SCALE}" />
         </geometry>
       </collision>
@@ -235,5 +235,5 @@
         <origin xyz="0 0 0" rpy="0 0 0" />
         <geometry>
-          <mesh filename="package://robotis_mini_description/meshes/DMF-B04(W).stl" scale="${STL_SCALE}" />
+          <mesh filename="package://robotis_mini_model/meshes/DMF-B04(W).stl" scale="${STL_SCALE}" />
         </geometry>
         <material name="White" />
@@ -249,5 +249,5 @@
       <collision>
         <geometry>
-          <mesh filename="package://robotis_mini_description/meshes/DMF-B04(W)_s.stl" scale="${STL_SCALE}" />
+          <mesh filename="package://robotis_mini_model/meshes/DMF-B04(W)_s.stl" scale="${STL_SCALE}" />
         </geometry>
       </collision>
@@ -265,5 +265,5 @@
         <origin xyz="0 0 0" rpy="0 0 0" />
         <geometry>
-          <mesh filename="package://robotis_mini_description/meshes/DMF-B05(W).stl" scale="${STL_SCALE}" />
+          <mesh filename="package://robotis_mini_model/meshes/DMF-B05(W).stl" scale="${STL_SCALE}" />
         </geometry>
         <material name="White" />
@@ -279,5 +279,5 @@
       <collision>
         <geometry>
-          <mesh filename="package://robotis_mini_description/meshes/DMF-B05(W)_s.stl" scale="${STL_SCALE}" />
+          <mesh filename="package://robotis_mini_model/meshes/DMF-B05(W)_s.stl" scale="${STL_SCALE}" />
         </geometry>
       </collision>
@@ -295,5 +295,5 @@
         <origin xyz="0 0 0" rpy="0 0 0" />
         <geometry>
-          <mesh filename="package://robotis_mini_description/meshes/DMF-B06(W).stl" scale="${STL_SCALE}" />
+          <mesh filename="package://robotis_mini_model/meshes/DMF-B06(W).stl" scale="${STL_SCALE}" />
         </geometry>
         <material name="White" />
@@ -309,5 +309,5 @@
       <collision>
         <geometry>
-          <mesh filename="package://robotis_mini_description/meshes/DMF-B06(W)_s.stl" scale="${STL_SCALE}" />
+          <mesh filename="package://robotis_mini_model/meshes/DMF-B06(W)_s.stl" scale="${STL_SCALE}" />
         </geometry>
       </collision>
@@ -325,5 +325,5 @@
         <origin xyz="0 0 0" rpy="0 0 0" />
         <geometry>
-          <mesh filename="package://robotis_mini_description/meshes/DMF-B07(GR).stl" scale="${STL_SCALE}" />
+          <mesh filename="package://robotis_mini_model/meshes/DMF-B07(GR).stl" scale="${STL_SCALE}" />
         </geometry>
         <material name="LightGrey" />
@@ -339,5 +339,5 @@
       <collision>
         <geometry>
-          <mesh filename="package://robotis_mini_description/meshes/DMF-B07(GR)_s.stl" scale="${STL_SCALE}" />
+          <mesh filename="package://robotis_mini_model/meshes/DMF-B07(GR)_s.stl" scale="${STL_SCALE}" />
         </geometry>
       </collision>
@@ -355,5 +355,5 @@
         <origin xyz="0 0 0" rpy="0 0 0" />
         <geometry>
-          <mesh filename="package://robotis_mini_description/meshes/DMF-F01(W).stl" scale="${STL_SCALE}" />
+          <mesh filename="package://robotis_mini_model/meshes/DMF-F01(W).stl" scale="${STL_SCALE}" />
         </geometry>
         <material name="White" />
@@ -369,5 +369,5 @@
       <collision>
         <geometry>
-          <mesh filename="package://robotis_mini_description/meshes/DMF-F01(W)_s.stl" scale="${STL_SCALE}" />
+          <mesh filename="package://robotis_mini_model/meshes/DMF-F01(W)_s.stl" scale="${STL_SCALE}" />
         </geometry>
       </collision>
@@ -385,5 +385,5 @@
         <origin xyz="0 0 0" rpy="0 0 0" />
         <geometry>
-          <mesh filename="package://robotis_mini_description/meshes/SPU-5(W).stl" scale="${STL_SCALE}" />
+          <mesh filename="package://robotis_mini_model/meshes/SPU-5(W).stl" scale="${STL_SCALE}" />
         </geometry>
         <material name="White" />
@@ -399,5 +399,5 @@
       <collision>
         <geometry>
-          <mesh filename="package://robotis_mini_description/meshes/SPU-5(W)_s.stl" scale="${STL_SCALE}" />
+          <mesh filename="package://robotis_mini_model/meshes/SPU-5(W)_s.stl" scale="${STL_SCALE}" />
         </geometry>
       </collision>
@@ -415,5 +415,5 @@
         <origin xyz="0 0 0" rpy="0 0 0" />
         <geometry>
-          <mesh filename="package://robotis_mini_description/meshes/SPD-3B3(W).stl" scale="${STL_SCALE}" />
+          <mesh filename="package://robotis_mini_model/meshes/SPD-3B3(W).stl" scale="${STL_SCALE}" />
         </geometry>
         <material name="White" />
@@ -429,5 +429,5 @@
       <collision>
         <geometry>
-          <mesh filename="package://robotis_mini_description/meshes/SPD-3B3(W)_s.stl" scale="${STL_SCALE}" />
+          <mesh filename="package://robotis_mini_model/meshes/SPD-3B3(W)_s.stl" scale="${STL_SCALE}" />
         </geometry>
       </collision>
@@ -445,5 +445,5 @@
         <origin xyz="0 0 0" rpy="0 0 0" />
         <geometry>
-          <mesh filename="package://robotis_mini_description/meshes/SPD-3B5(W).stl" scale="${STL_SCALE}" />
+          <mesh filename="package://robotis_mini_model/meshes/SPD-3B5(W).stl" scale="${STL_SCALE}" />
         </geometry>
         <material name="White" />
@@ -459,5 +459,5 @@
       <collision>
         <geometry>
-          <mesh filename="package://robotis_mini_description/meshes/SPD-3B5(W)_s.stl" scale="${STL_SCALE}" />
+          <mesh filename="package://robotis_mini_model/meshes/SPD-3B5(W)_s.stl" scale="${STL_SCALE}" />
         </geometry>
       </collision>
@@ -475,5 +475,5 @@
         <origin xyz="0 0 0" rpy="0 0 0" />
         <geometry>
-          <mesh filename="package://robotis_mini_description/meshes/SPD-3B7(W).stl" scale="${STL_SCALE}" />
+          <mesh filename="package://robotis_mini_model/meshes/SPD-3B7(W).stl" scale="${STL_SCALE}" />
         </geometry>
         <material name="White" />
@@ -489,5 +489,5 @@
       <collision>
         <geometry>
-          <mesh filename="package://robotis_mini_description/meshes/SPD-3B7(W)_s.stl" scale="${STL_SCALE}" />
+          <mesh filename="package://robotis_mini_model/meshes/SPD-3B7(W)_s.stl" scale="${STL_SCALE}" />
         </geometry>
       </collision>
@@ -505,5 +505,5 @@
         <origin xyz="0 0 0" rpy="0 0 0" />
         <geometry>
-          <mesh filename="package://robotis_mini_description/meshes/SPD-4B5(W).stl" scale="${STL_SCALE}" />
+          <mesh filename="package://robotis_mini_model/meshes/SPD-4B5(W).stl" scale="${STL_SCALE}" />
         </geometry>
         <material name="White" />
@@ -519,5 +519,5 @@
       <collision>
         <geometry>
-          <mesh filename="package://robotis_mini_description/meshes/SPD-4B5(W)_s.stl" scale="${STL_SCALE}" />
+          <mesh filename="package://robotis_mini_model/meshes/SPD-4B5(W)_s.stl" scale="${STL_SCALE}" />
         </geometry>
       </collision>
@@ -535,5 +535,5 @@
         <origin xyz="0 0 0" rpy="0 0 0" />
         <geometry>
-          <mesh filename="package://robotis_mini_description/meshes/SPD-7V4(W).stl" scale="${STL_SCALE}" />
+          <mesh filename="package://robotis_mini_model/meshes/SPD-7V4(W).stl" scale="${STL_SCALE}" />
         </geometry>
         <material name="White" />
@@ -549,5 +549,5 @@
       <collision>
         <geometry>
-          <mesh filename="package://robotis_mini_description/meshes/SPD-7V4(W)_s.stl" scale="${STL_SCALE}" />
+          <mesh filename="package://robotis_mini_model/meshes/SPD-7V4(W)_s.stl" scale="${STL_SCALE}" />
         </geometry>
       </collision>
@@ -565,5 +565,5 @@
         <origin xyz="0 0 0" rpy="0 0 0" />
         <geometry>
-          <mesh filename="package://robotis_mini_description/meshes/SPL-2B2(W).stl" scale="${STL_SCALE}" />
+          <mesh filename="package://robotis_mini_model/meshes/SPL-2B2(W).stl" scale="${STL_SCALE}" />
         </geometry>
         <material name="White" />
@@ -579,5 +579,5 @@
       <collision>
         <geometry>
-          <mesh filename="package://robotis_mini_description/meshes/SPL-2B2(W)_s.stl" scale="${STL_SCALE}" />
+          <mesh filename="package://robotis_mini_model/meshes/SPL-2B2(W)_s.stl" scale="${STL_SCALE}" />
         </geometry>
       </collision>
@@ -595,5 +595,5 @@
         <origin xyz="0 0 0" rpy="0 0 0" />
         <geometry>
-          <mesh filename="package://robotis_mini_description/meshes/SPO-5(GR).stl" scale="${STL_SCALE}" />
+          <mesh filename="package://robotis_mini_model/meshes/SPO-5(GR).stl" scale="${STL_SCALE}" />
         </geometry>
         <material name="LightGrey" />
@@ -609,5 +609,5 @@
       <collision>
         <geometry>
-          <mesh filename="package://robotis_mini_description/meshes/SPO-5(GR)_s.stl" scale="${STL_SCALE}" />
+          <mesh filename="package://robotis_mini_model/meshes/SPO-5(GR)_s.stl" scale="${STL_SCALE}" />
         </geometry>
       </collision>
@@ -650,5 +650,5 @@
         <origin xyz="0 0 0" rpy="0 0 0" />
         <geometry>
-          <mesh filename="package://robotis_mini_description/meshes/XL-320D.stl" scale="${STL_SCALE}" />
+          <mesh filename="package://robotis_mini_model/meshes/XL-320D.stl" scale="${STL_SCALE}" />
         </geometry>
         <material name="Grey" />
@@ -664,5 +664,5 @@
       <collision>
         <geometry>
-          <mesh filename="package://robotis_mini_description/meshes/XL-320D.stl" scale="${STL_SCALE}" />
+          <mesh filename="package://robotis_mini_model/meshes/XL-320D.stl" scale="${STL_SCALE}" />
         </geometry>
       </collision>

File: robotis_mini_model/urdf/robotis_mini.urdf.xacro (robot description, xacro)
@@ -5,12 +5,12 @@
        xmlns:xacro="http://www.ros.org/wiki/xacro"
        name="robotis_mini" >
-  <xacro:include filename="$(find-pkg-share robotis_mini_model)/urdf/materials.urdf.xacro" />
-  <xacro:include filename="$(find-pkg-share robotis_mini_model)/urdf/common.urdf.xacro" />
-  <xacro:include filename="$(find-pkg-share robotis_mini_model)/urdf/servo.urdf.xacro" />
-  <xacro:include filename="$(find-pkg-share robotis_mini_model)/urdf/base.urdf.xacro" />
-  <xacro:include filename="$(find-pkg-share robotis_mini_model)/urdf/body.urdf.xacro" />
-  <xacro:include filename="$(find-pkg-share robotis_mini_model)/urdf/arm.urdf.xacro" />
-  <xacro:include filename="$(find-pkg-share robotis_mini_model)/urdf/hand.urdf.xacro" />
-  <xacro:include filename="$(find-pkg-share robotis_mini_model)/urdf/leg.urdf.xacro" />
+  <xacro:include filename="materials.urdf.xacro" />
+  <xacro:include filename="common.urdf.xacro" />
+  <xacro:include filename="servo.urdf.xacro" />
+  <xacro:include filename="base.urdf.xacro" />
+  <xacro:include filename="body.urdf.xacro" />
+  <xacro:include filename="arm.urdf.xacro" />
+  <xacro:include filename="hand.urdf.xacro" />
+  <xacro:include filename="leg.urdf.xacro" />
   <xacro:robotis_mini_base name="base"/>
   <!-- <xacro:robotis_mini_body2 parent="base_link" />

Commit message: SImplify xl-320d motor

File: robotis_mini_model/urdf/common.urdf.xacro (robot description, xacro)
@@ -664,5 +664,5 @@
       <collision>
         <geometry>
-          <mesh filename="package://robotis_mini_model/meshes/XL-320D.stl" scale="${STL_SCALE}" />
+          <mesh filename="package://robotis_mini_model/meshes/XL-320D_s.stl" scale="${STL_SCALE}" />
         </geometry>
       </collision>

File: robotis_mini_model/urdf/robotis_mini.urdf (robot description, URDF)
Before this commit: robot robotis_mini, 105 links, 104 joints
Links:
- link l_ankle_link: geometry collision mesh filename=package://robotis_mini_model/meshes/XL-320D_s.stl scale=0.001 0.001 0.001; visual mesh filename=package://robotis_mini_model/meshes/XL-320D.stl scale=0.001 0.001 0.001
- link l_biceps_link: geometry collision mesh filename=package://robotis_mini_model/meshes/XL-320D_s.stl scale=0.001 0.001 0.001; visual mesh filename=package://robotis_mini_model/meshes/XL-320D.stl scale=0.001 0.001 0.001
- link l_elbow_link: geometry collision mesh filename=package://robotis_mini_model/meshes/XL-320D_s.stl scale=0.001 0.001 0.001; visual mesh filename=package://robotis_mini_model/meshes/XL-320D.stl scale=0.001 0.001 0.001
- link l_foot_link: geometry collision mesh filename=package://robotis_mini_model/meshes/XL-320D_s.stl scale=0.001 0.001 0.001; visual mesh filename=package://robotis_mini_model/meshes/XL-320D.stl scale=0.001 0.001 0.001
- link l_hip_servo_link: geometry collision mesh filename=package://robotis_mini_model/meshes/XL-320D_s.stl scale=0.001 0.001 0.001; visual mesh filename=package://robotis_mini_model/meshes/XL-320D.stl scale=0.001 0.001 0.001
- link l_knee_servo_link: geometry collision mesh filename=package://robotis_mini_model/meshes/XL-320D_s.stl scale=0.001 0.001 0.001; visual mesh filename=package://robotis_mini_model/meshes/XL-320D.stl scale=0.001 0.001 0.001
- link l_shoulder_servo_link: geometry collision mesh filename=package://robotis_mini_model/meshes/XL-320D_s.stl scale=0.001 0.001 0.001; visual mesh filename=package://robotis_mini_model/meshes/XL-320D.stl scale=0.001 0.001 0.001
- link l_thigh_servo_link: geometry collision mesh filename=package://robotis_mini_model/meshes/XL-320D_s.stl scale=0.001 0.001 0.001; visual mesh filename=package://robotis_mini_model/meshes/XL-320D.stl scale=0.001 0.001 0.001
- link neck_link: geometry collision mesh filename=package://robotis_mini_model/meshes/XL-320D_s.stl scale=0.001 0.001 0.001; visual mesh filename=package://robotis_mini_model/meshes/XL-320D.stl scale=0.001 0.001 0.001
- link r_ankle_link: geometry collision mesh filename=package://robotis_mini_model/meshes/XL-320D_s.stl scale=0.001 0.001 0.001; visual mesh filename=package://robotis_mini_model/meshes/XL-320D.stl scale=0.001 0.001 0.001
- link r_biceps_link: geometry collision mesh filename=package://robotis_mini_model/meshes/XL-320D_s.stl scale=0.001 0.001 0.001; visual mesh filename=package://robotis_mini_model/meshes/XL-320D.stl scale=0.001 0.001 0.001
- link r_elbow_link: geometry collision mesh filename=package://robotis_mini_model/meshes/XL-320D_s.stl scale=0.001 0.001 0.001; visual mesh filename=package://robotis_mini_model/meshes/XL-320D.stl scale=0.001 0.001 0.001
- link r_foot_link: geometry collision mesh filename=package://robotis_mini_model/meshes/XL-320D_s.stl scale=0.001 0.001 0.001; visual mesh filename=package://robotis_mini_model/meshes/XL-320D.stl scale=0.001 0.001 0.001
- link r_hip_servo_link: geometry collision mesh filename=package://robotis_mini_model/meshes/XL-320D_s.stl scale=0.001 0.001 0.001; visual mesh filename=package://robotis_mini_model/meshes/XL-320D.stl scale=0.001 0.001 0.001
- link r_knee_servo_link: geometry collision mesh filename=package://robotis_mini_model/meshes/XL-320D_s.stl scale=0.001 0.001 0.001; visual mesh filename=package://robotis_mini_model/meshes/XL-320D.stl scale=0.001 0.001 0.001
- link r_shoulder_servo_link: geometry collision mesh filename=package://robotis_mini_model/meshes/XL-320D_s.stl scale=0.001 0.001 0.001; visual mesh filename=package://robotis_mini_model/meshes/XL-320D.stl scale=0.001 0.001 0.001
- link r_thigh_servo_link: geometry collision mesh filename=package://robotis_mini_model/meshes/XL-320D_s.stl scale=0.001 0.001 0.001; visual mesh filename=package://robotis_mini_model/meshes/XL-320D.stl scale=0.001 0.001 0.001
