Commit message: Disable all small parts.

File: robotis_mini_model/urdf/common.urdf.xacro (robot description, xacro)
@@ -159,5 +159,6 @@
       <collision>
         <geometry>
-          <mesh filename="package://robotis_mini_model/meshes/DMF-B01(W)_s.stl" scale="${STL_SCALE}" />
+          <!--<mesh filename="package://robotis_mini_model/meshes/DMF-B01(W)_s.stl" scale="${STL_SCALE}" />-->
+          <sphere radius="0" />
         </geometry>
       </collision>
@@ -189,5 +190,6 @@
       <collision>
         <geometry>
-          <mesh filename="package://robotis_mini_model/meshes/DMB-B02(W)_s.stl" scale="${STL_SCALE}" />
+          <!--<mesh filename="package://robotis_mini_model/meshes/DMB-B02(W)_s.stl" scale="${STL_SCALE}" />-->
+          <sphere radius="0" />
         </geometry>
       </collision>
@@ -219,5 +221,6 @@
       <collision>
         <geometry>
-          <mesh filename="package://robotis_mini_model/meshes/DMF-B03(W)_s.stl" scale="${STL_SCALE}" />
+          <!--<mesh filename="package://robotis_mini_model/meshes/DMF-B03(W)_s.stl" scale="${STL_SCALE}" />-->
+          <sphere radius="0" />
         </geometry>
       </collision>
@@ -249,5 +252,6 @@
       <collision>
         <geometry>
-          <mesh filename="package://robotis_mini_model/meshes/DMF-B04(W)_s.stl" scale="${STL_SCALE}" />
+          <!--<mesh filename="package://robotis_mini_model/meshes/DMF-B04(W)_s.stl" scale="${STL_SCALE}" />-->
+          <sphere radius="0" />
         </geometry>
       </collision>
@@ -279,5 +283,6 @@
       <collision>
         <geometry>
-          <mesh filename="package://robotis_mini_model/meshes/DMF-B05(W)_s.stl" scale="${STL_SCALE}" />
+          <!--<mesh filename="package://robotis_mini_model/meshes/DMF-B05(W)_s.stl" scale="${STL_SCALE}" />-->
+          <sphere radius="0" />
         </geometry>
       </collision>
@@ -309,5 +314,6 @@
       <collision>
         <geometry>
-          <mesh filename="package://robotis_mini_model/meshes/DMF-B06(W)_s.stl" scale="${STL_SCALE}" />
+          <!--<mesh filename="package://robotis_mini_model/meshes/DMF-B06(W)_s.stl" scale="${STL_SCALE}" />-->
+          <sphere radius="0" />
         </geometry>
       </collision>
@@ -339,5 +345,6 @@
       <collision>
         <geometry>
-          <mesh filename="package://robotis_mini_model/meshes/DMF-B07(GR)_s.stl" scale="${STL_SCALE}" />
+          <!--<mesh filename="package://robotis_mini_model/meshes/DMF-B07(GR)_s.stl" scale="${STL_SCALE}" />-->
+          <sphere radius="0" />
         </geometry>
       </collision>
@@ -369,5 +376,6 @@
       <collision>
         <geometry>
-          <mesh filename="package://robotis_mini_model/meshes/DMF-F01(W)_s.stl" scale="${STL_SCALE}" />
+          <!--<mesh filename="package://robotis_mini_model/meshes/DMF-F01(W)_s.stl" scale="${STL_SCALE}" />-->
+          <sphere radius="0" />
         </geometry>
       </collision>
@@ -399,5 +407,6 @@
       <collision>
         <geometry>
-          <mesh filename="package://robotis_mini_model/meshes/SPU-5(W)_s.stl" scale="${STL_SCALE}" />
+          <!--<mesh filename="package://robotis_mini_model/meshes/SPU-5(W)_s.stl" scale="${STL_SCALE}" />-->
+          <sphere radius="0" />
         </geometry>
       </collision>
@@ -429,5 +438,6 @@
       <collision>
         <geometry>
-          <mesh filename="package://robotis_mini_model/meshes/SPD-3B3(W)_s.stl" scale="${STL_SCALE}" />
+          <!--<mesh filename="package://robotis_mini_model/meshes/SPD-3B3(W)_s.stl" scale="${STL_SCALE}" />-->
+          <sphere radius="0" />
         </geometry>
       </collision>
@@ -459,5 +469,6 @@
       <collision>
         <geometry>
-          <mesh filename="package://robotis_mini_model/meshes/SPD-3B5(W)_s.stl" scale="${STL_SCALE}" />
+          <!--<mesh filename="package://robotis_mini_model/meshes/SPD-3B5(W)_s.stl" scale="${STL_SCALE}" />-->
+          <sphere radius="0" />
         </geometry>
       </collision>
@@ -489,5 +500,6 @@
       <collision>
         <geometry>
-          <mesh filename="package://robotis_mini_model/meshes/SPD-3B7(W)_s.stl" scale="${STL_SCALE}" />
+          <!--<mesh filename="package://robotis_mini_model/meshes/SPD-3B7(W)_s.stl" scale="${STL_SCALE}" />-->
+          <sphere radius="0" />
         </geometry>
       </collision>
@@ -519,5 +531,6 @@
       <collision>
         <geometry>
-          <mesh filename="package://robotis_mini_model/meshes/SPD-4B5(W)_s.stl" scale="${STL_SCALE}" />
+          <!--<mesh filename="package://robotis_mini_model/meshes/SPD-4B5(W)_s.stl" scale="${STL_SCALE}" />-->
+          <sphere radius="0" />
         </geometry>
       </collision>
@@ -549,5 +562,6 @@
       <collision>
         <geometry>
-          <mesh filename="package://robotis_mini_model/meshes/SPD-7V4(W)_s.stl" scale="${STL_SCALE}" />
+          <!--<mesh filename="package://robotis_mini_model/meshes/SPD-7V4(W)_s.stl" scale="${STL_SCALE}" />-->
+          <sphere radius="0" />
         </geometry>
       </collision>
@@ -579,5 +593,6 @@
       <collision>
         <geometry>
-          <mesh filename="package://robotis_mini_model/meshes/SPL-2B2(W)_s.stl" scale="${STL_SCALE}" />
+          <!--<mesh filename="package://robotis_mini_model/meshes/SPL-2B2(W)_s.stl" scale="${STL_SCALE}" />-->
+          <sphere radius="0" />
         </geometry>
       </collision>
@@ -609,5 +624,6 @@
       <collision>
         <geometry>
-          <mesh filename="package://robotis_mini_model/meshes/SPO-5(GR)_s.stl" scale="${STL_SCALE}" />
+          <!--<mesh filename="package://robotis_mini_model/meshes/SPO-5(GR)_s.stl" scale="${STL_SCALE}" />-->
+          <sphere radius="0" />
         </geometry>
       </collision>
@@ -664,5 +680,6 @@
       <collision>
         <geometry>
-          <mesh filename="package://robotis_mini_model/meshes/XL-320D_s.stl" scale="${STL_SCALE}" />
+          <!--<mesh filename="package://robotis_mini_model/meshes/XL-320D_s.stl" scale="${STL_SCALE}" />-->
+          <sphere radius="0" />
         </geometry>
       </collision>
