Commit message: Regenerate urdf with small part as balls

File: robotis_mini_model/urdf/robotis_mini.urdf (robot description, URDF)
Before this commit: robot robotis_mini, 105 links, 104 joints
Links:
- link body_head_link: geometry collision sphere radius=0; visual mesh filename=package://robotis_mini_model/meshes/DMF-F01(W).stl scale=0.001 0.001 0.001
- link body_skeleton_link: geometry collision sphere radius=0; visual mesh filename=package://robotis_mini_model/meshes/DMB-B02(W).stl scale=0.001 0.001 0.001
- link body_torso_link: geometry collision sphere radius=0; visual mesh filename=package://robotis_mini_model/meshes/DMF-B01(W).stl scale=0.001 0.001 0.001
- link l_achiles_link: geometry collision sphere radius=0; visual mesh filename=package://robotis_mini_model/meshes/SPD-3B7(W).stl scale=0.001 0.001 0.001
- link l_ankle_link: geometry collision sphere radius=0; visual mesh filename=package://robotis_mini_model/meshes/XL-320D.stl scale=0.001 0.001 0.001
- link l_ankle_spo_link: geometry collision sphere radius=0; visual mesh filename=package://robotis_mini_model/meshes/SPO-5(GR).stl scale=0.001 0.001 0.001
- link l_biceps_anchor_link: geometry collision sphere radius=0; visual mesh filename=package://robotis_mini_model/meshes/DMF-B03(W).stl scale=0.001 0.001 0.001
- link l_biceps_link: geometry collision sphere radius=0; visual mesh filename=package://robotis_mini_model/meshes/XL-320D.stl scale=0.001 0.001 0.001
- link l_biceps_spo_link: geometry collision sphere radius=0; visual mesh filename=package://robotis_mini_model/meshes/SPO-5(GR).stl scale=0.001 0.001 0.001
- link l_elbow_link: geometry collision sphere radius=0; visual mesh filename=package://robotis_mini_model/meshes/XL-320D.stl scale=0.001 0.001 0.001
- link l_elbow_spo_link: geometry collision sphere radius=0; visual mesh filename=package://robotis_mini_model/meshes/SPO-5(GR).stl scale=0.001 0.001 0.001
- link l_foot_anchor_link: geometry collision sphere radius=0; visual mesh filename=package://robotis_mini_model/meshes/SPD-7V4(W).stl scale=0.001 0.001 0.001
- link l_foot_link: geometry collision sphere radius=0; visual mesh filename=package://robotis_mini_model/meshes/XL-320D.stl scale=0.001 0.001 0.001
- link l_forefoot_link: geometry collision sphere radius=0; visual mesh filename=package://robotis_mini_model/meshes/DMF-B06(W).stl scale=0.001 0.001 0.001
- link l_groin_link: geometry collision sphere radius=0; visual mesh filename=package://robotis_mini_model/meshes/SPD-7V4(W).stl scale=0.001 0.001 0.001
- link l_hand_back_link: geometry collision sphere radius=0; visual mesh filename=package://robotis_mini_model/meshes/SPD-4B5(W).stl scale=0.001 0.001 0.001
- link l_hand_base_link: geometry collision sphere radius=0; visual mesh filename=package://robotis_mini_model/meshes/SPD-3B5(W).stl scale=0.001 0.001 0.001
- link l_hand_fingers_ext1_link: geometry collision sphere radius=0; visual mesh filename=package://robotis_mini_model/meshes/SPL-2B2(W).stl scale=0.001 0.001 0.001
- link l_hand_fingers_ext2_link: geometry collision sphere radius=0; visual mesh filename=package://robotis_mini_model/meshes/SPL-2B2(W).stl scale=0.001 0.001 0.001
- link l_hand_fingers_int1_link: geometry collision sphere radius=0; visual mesh filename=package://robotis_mini_model/meshes/SPL-2B2(W).stl scale=0.001 0.001 0.001
- link l_hand_fingers_int2_link: geometry collision sphere radius=0; visual mesh filename=package://robotis_mini_model/meshes/SPL-2B2(W).stl scale=0.001 0.001 0.001
- link l_hand_palm_anchor1_link: geometry collision sphere radius=0; visual mesh filename=package://robotis_mini_model/meshes/SPL-2B2(W).stl scale=0.001 0.001 0.001
- link l_hand_palm_anchor2_link: geometry collision sphere radius=0; visual mesh filename=package://robotis_mini_model/meshes/SPL-2B2(W).stl scale=0.001 0.001 0.001
- link l_hand_palm_link: geometry collision sphere radius=0; visual mesh filename=package://robotis_mini_model/meshes/SPD-3B5(W).stl scale=0.001 0.001 0.001
- link l_hand_thumb_link: geometry collision sphere radius=0; visual mesh filename=package://robotis_mini_model/meshes/SPL-2B2(W).stl scale=0.001 0.001 0.001
- link l_hand_wrist1_link: geometry collision sphere radius=0; visual mesh filename=package://robotis_mini_model/meshes/SPO-5(GR).stl scale=0.001 0.001 0.001
- link l_hand_wrist2_link: geometry collision sphere radius=0; visual mesh filename=package://robotis_mini_model/meshes/SPO-5(GR).stl scale=0.001 0.001 0.001
- link l_hip_anchor_link: geometry collision sphere radius=0; visual mesh filename=package://robotis_mini_model/meshes/SPU-5(W).stl scale=0.001 0.001 0.001
- link l_hip_servo_link: geometry collision sphere radius=0; visual mesh filename=package://robotis_mini_model/meshes/XL-320D.stl scale=0.001 0.001 0.001
- link l_knee_servo_link: geometry collision sphere radius=0; visual mesh filename=package://robotis_mini_model/meshes/XL-320D.stl scale=0.001 0.001 0.001
- link l_knee_spo_link: geometry collision sphere radius=0; visual mesh filename=package://robotis_mini_model/meshes/SPO-5(GR).stl scale=0.001 0.001 0.001
- link l_lower_arm_link: geometry collision sphere radius=0; visual mesh filename=package://robotis_mini_model/meshes/SPU-5(W).stl scale=0.001 0.001 0.001
- link l_lower_leg_link: geometry collision sphere radius=0; visual mesh filename=package://robotis_mini_model/meshes/DMF-B05(W).stl scale=0.001 0.001 0.001
- link l_shoulder_anchor_link: geometry collision sphere radius=0; visual mesh filename=package://robotis_mini_model/meshes/SPU-5(W).stl scale=0.001 0.001 0.001
- link l_shoulder_servo_link: geometry collision sphere radius=0; visual mesh filename=package://robotis_mini_model/meshes/XL-320D.stl scale=0.001 0.001 0.001
- link l_sole_link: geometry collision sphere radius=0; visual mesh filename=package://robotis_mini_model/meshes/DMF-B07(GR).stl scale=0.001 0.001 0.001
- link l_thigh_anchor_link: geometry collision sphere radius=0; visual mesh filename=package://robotis_mini_model/meshes/SPD-3B5(W).stl scale=0.001 0.001 0.001
- link l_thigh_servo_link: geometry collision sphere radius=0; visual mesh filename=package://robotis_mini_model/meshes/XL-320D.stl scale=0.001 0.001 0.001
- link l_thigh_spo_link: geometry collision sphere radius=0; visual mesh filename=package://robotis_mini_model/meshes/SPO-5(GR).stl scale=0.001 0.001 0.001
- link l_thigh_top_link: geometry collision sphere radius=0; visual mesh filename=package://robotis_mini_model/meshes/SPU-5(W).stl scale=0.001 0.001 0.001
- link l_upper_arm_link: geometry collision sphere radius=0; visual mesh filename=package://robotis_mini_model/meshes/DMF-B04(W).stl scale=0.001 0.001 0.001
- link l_upper_leg_link: geometry collision sphere radius=0; visual mesh filename=package://robotis_mini_model/meshes/DMF-B04(W).stl scale=0.001 0.001 0.001
- link l_wrist_anchor_link: geometry collision sphere radius=0; visual mesh filename=package://robotis_mini_model/meshes/SPD-3B3(W).stl scale=0.001 0.001 0.001
- link neck_link: geometry collision sphere radius=0; visual mesh filename=package://robotis_mini_model/meshes/XL-320D.stl scale=0.001 0.001 0.001
- link r_achiles_link: geometry collision sphere radius=0; visual mesh filename=package://robotis_mini_model/meshes/SPD-3B7(W).stl scale=0.001 0.001 0.001
- link r_ankle_link: geometry collision sphere radius=0; visual mesh filename=package://robotis_mini_model/meshes/XL-320D.stl scale=0.001 0.001 0.001
- link r_ankle_spo_link: geometry collision sphere radius=0; visual mesh filename=package://robotis_mini_model/meshes/SPO-5(GR).stl scale=0.001 0.001 0.001
- link r_biceps_anchor_link: geometry collision sphere radius=0; visual mesh filename=package://robotis_mini_model/meshes/DMF-B03(W).stl scale=0.001 0.001 0.001
- link r_biceps_link: geometry collision sphere radius=0; visual mesh filename=package://robotis_mini_model/meshes/XL-320D.stl scale=0.001 0.001 0.001
- link r_biceps_spo_link: geometry collision sphere radius=0; visual mesh filename=package://robotis_mini_model/meshes/SPO-5(GR).stl scale=0.001 0.001 0.001
- link r_elbow_link: geometry collision sphere radius=0; visual mesh filename=package://robotis_mini_model/meshes/XL-320D.stl scale=0.001 0.001 0.001
- link r_elbow_spo_link: geometry collision sphere radius=0; visual mesh filename=package://robotis_mini_model/meshes/SPO-5(GR).stl scale=0.001 0.001 0.001
- link r_foot_anchor_link: geometry collision sphere radius=0; visual mesh filename=package://robotis_mini_model/meshes/SPD-7V4(W).stl scale=0.001 0.001 0.001
- link r_foot_link: geometry collision sphere radius=0; visual mesh filename=package://robotis_mini_model/meshes/XL-320D.stl scale=0.001 0.001 0.001
- link r_forefoot_link: geometry collision sphere radius=0; visual mesh filename=package://robotis_mini_model/meshes/DMF-B06(W).stl scale=0.001 0.001 0.001
- link r_groin_link: geometry collision sphere radius=0; visual mesh filename=package://robotis_mini_model/meshes/SPD-7V4(W).stl scale=0.001 0.001 0.001
- link r_hand_back_link: geometry collision sphere radius=0; visual mesh filename=package://robotis_mini_model/meshes/SPD-4B5(W).stl scale=0.001 0.001 0.001
- link r_hand_base_link: geometry collision sphere radius=0; visual mesh filename=package://robotis_mini_model/meshes/SPD-3B5(W).stl scale=0.001 0.001 0.001
- link r_hand_fingers_ext1_link: geometry collision sphere radius=0; visual mesh filename=package://robotis_mini_model/meshes/SPL-2B2(W).stl scale=0.001 0.001 0.001
- link r_hand_fingers_ext2_link: geometry collision sphere radius=0; visual mesh filename=package://robotis_mini_model/meshes/SPL-2B2(W).stl scale=0.001 0.001 0.001
- link r_hand_fingers_int1_link: geometry collision sphere radius=0; visual mesh filename=package://robotis_mini_model/meshes/SPL-2B2(W).stl scale=0.001 0.001 0.001
- link r_hand_fingers_int2_link: geometry collision sphere radius=0; visual mesh filename=package://robotis_mini_model/meshes/SPL-2B2(W).stl scale=0.001 0.001 0.001
- link r_hand_palm_anchor1_link: geometry collision sphere radius=0; visual mesh filename=package://robotis_mini_model/meshes/SPL-2B2(W).stl scale=0.001 0.001 0.001
- link r_hand_palm_anchor2_link: geometry collision sphere radius=0; visual mesh filename=package://robotis_mini_model/meshes/SPL-2B2(W).stl scale=0.001 0.001 0.001
- link r_hand_palm_link: geometry collision sphere radius=0; visual mesh filename=package://robotis_mini_model/meshes/SPD-3B5(W).stl scale=0.001 0.001 0.001
- link r_hand_thumb_link: geometry collision sphere radius=0; visual mesh filename=package://robotis_mini_model/meshes/SPL-2B2(W).stl scale=0.001 0.001 0.001
- link r_hand_wrist1_link: geometry collision sphere radius=0; visual mesh filename=package://robotis_mini_model/meshes/SPO-5(GR).stl scale=0.001 0.001 0.001
- link r_hand_wrist2_link: geometry collision sphere radius=0; visual mesh filename=package://robotis_mini_model/meshes/SPO-5(GR).stl scale=0.001 0.001 0.001
- link r_hip_anchor_link: geometry collision sphere radius=0; visual mesh filename=package://robotis_mini_model/meshes/SPU-5(W).stl scale=0.001 0.001 0.001
- link r_hip_servo_link: geometry collision sphere radius=0; visual mesh filename=package://robotis_mini_model/meshes/XL-320D.stl scale=0.001 0.001 0.001
- link r_knee_servo_link: geometry collision sphere radius=0; visual mesh filename=package://robotis_mini_model/meshes/XL-320D.stl scale=0.001 0.001 0.001
- link r_knee_spo_link: geometry collision sphere radius=0; visual mesh filename=package://robotis_mini_model/meshes/SPO-5(GR).stl scale=0.001 0.001 0.001
- link r_lower_arm_link: geometry collision sphere radius=0; visual mesh filename=package://robotis_mini_model/meshes/SPU-5(W).stl scale=0.001 0.001 0.001
- link r_lower_leg_link: geometry collision sphere radius=0; visual mesh filename=package://robotis_mini_model/meshes/DMF-B05(W).stl scale=0.001 0.001 0.001
- link r_shoulder_anchor_link: geometry collision sphere radius=0; visual mesh filename=package://robotis_mini_model/meshes/SPU-5(W).stl scale=0.001 0.001 0.001
- link r_shoulder_servo_link: geometry collision sphere radius=0; visual mesh filename=package://robotis_mini_model/meshes/XL-320D.stl scale=0.001 0.001 0.001
- link r_sole_link: geometry collision sphere radius=0; visual mesh filename=package://robotis_mini_model/meshes/DMF-B07(GR).stl scale=0.001 0.001 0.001
- link r_thigh_anchor_link: geometry collision sphere radius=0; visual mesh filename=package://robotis_mini_model/meshes/SPD-3B5(W).stl scale=0.001 0.001 0.001
- link r_thigh_servo_link: geometry collision sphere radius=0; visual mesh filename=package://robotis_mini_model/meshes/XL-320D.stl scale=0.001 0.001 0.001
- link r_thigh_spo_link: geometry collision sphere radius=0; visual mesh filename=package://robotis_mini_model/meshes/SPO-5(GR).stl scale=0.001 0.001 0.001
- link r_thigh_top_link: geometry collision sphere radius=0; visual mesh filename=package://robotis_mini_model/meshes/SPU-5(W).stl scale=0.001 0.001 0.001
- link r_upper_arm_link: geometry collision sphere radius=0; visual mesh filename=package://robotis_mini_model/meshes/DMF-B04(W).stl scale=0.001 0.001 0.001
- link r_upper_leg_link: geometry collision sphere radius=0; visual mesh filename=package://robotis_mini_model/meshes/DMF-B04(W).stl scale=0.001 0.001 0.001
- link r_wrist_anchor_link: geometry collision sphere radius=0; visual mesh filename=package://robotis_mini_model/meshes/SPD-3B3(W).stl scale=0.001 0.001 0.001
